Commit message: Finished A.3. Set up yaml file and finished setting up URDF to follow xacro format. Began on A.4 and changed color to be xacro. Note: the common_properties urdf contains only common colors that can be set for the robot.

File: nuturtle_description/urdf/common_properties.urdf.xacro (robot description, xacro)
@@ -1,8 +1,8 @@
 <?xml version="1.0" ?>
 <robot name="xacro_properties" xmlns:xacro="http://ros.org/wiki/xacro">
-<!-- This document has been modified from the original URDF provided by ROBOTIS.
-This modifications allow this URDF to be launched solely from this package,
-removing all dependencies on ROBOTIS turtlebot3 open-source package.Furthermore,
-this document has been modified to use xacro. -->
+  <!-- This document has been modified from the original URDF provided by ROBOTIS.
+  This modifications allow this URDF to be launched solely from this package,
+  removing all dependencies on ROBOTIS turtlebot3 open-source package.Furthermore,
+  this document has been modified to use xacro. -->
   <!-- Init colour -->
   <material name="black">

File: nuturtle_description/urdf/turtlebot3_burger.urdf.xacro (robot description, xacro)
@@ -1,18 +1,23 @@
 <?xml version="1.0" ?>
 <robot name="nuturtle" xmlns:xacro="http://ros.org/wiki/xacro">
-<!-- This document has been modified from the original URDF provided by ROBOTIS.
-This modifications allow this URDF to be launched solely from this package,
-removing all dependencies on ROBOTIS turtlebot3 open-source package.Furthermore,
-this document has been modified to use xacro. -->
+  <!-- This document has been modified from the original URDF provided by ROBOTIS.
+  This modifications allow this URDF to be launched solely from this package,
+  removing all dependencies on ROBOTIS turtlebot3 open-source package.Furthermore,
+  this document has been modified to use xacro. -->
   <!-- Loading in the YAML Configurations -->
-  <!-- <xacro:property name="yaml_file" value="$(find nuturtle_description)/config/diff_params.yaml"/>
-  <xacro:property name="config" value="${xacro.load_yaml(yaml_file)}"/> -->
+  <xacro:property name="yaml_file" value="$(find nuturtle_description)/config/diff_params.yaml"/>
+  <xacro:property name="config" value="${xacro.load_yaml(yaml_file)}"/>
   <!-- Define properties from YAML keys -->
-  <!-- <xacro:property name="platform_height" value="${config['/**']['ros__parameters']['platform_height']}"/>
-  <xacro:property name="wheel_radius" value="${config['/**']['ros__parameters']['wheel_radius']}"/> -->
+  <xacro:property name="wheel_radius" value="${config['/**']['ros__parameters']['wheel_radius']}"/>
+  <xacro:property name="track_width" value="${config['/**']['ros__parameters']['track_width']}"/>
+  <xacro:property name="collision_radius" value="${config['/**']['ros__parameters']['collision_radius']}"/>
+  <!-- Define color property from Launch File -->
+  <!-- <xacro:property name="color" value="${config['/**']['ros__parameters']['color']}"/> -->
   <!--Load in the Xacros created to establish the colors of the nuturtle-->
   <xacro:include filename="$(find nuturtle_description)/urdf/common_properties.urdf.xacro"/>
+  <!-- Set the namespace of the robot -->
   <xacro:arg name="namespace" default=""/>
   <xacro:property name="namespace" value="$(arg namespace)"/>
+ <!-- Use the Xacros to build the URDF-->
   <link name="${namespace}base_footprint"/>
   <joint name="${namespace}base_joint" type="fixed">
@@ -21,4 +26,5 @@
     <origin xyz="0.0 0.0 0.010" rpy="0 0 0"/>
   </joint>
+  <!-- Set the BaseLink -->
   <link name="${namespace}base_link">
     <visual>
@@ -27,10 +33,10 @@
         <mesh filename="package://nuturtle_description/meshes/burger_base.stl" scale="0.001 0.001 0.001"/>
       </geometry>
-      <material name="light_black"/>
+      <material name="${color}"/>
     </visual>
     <collision>
       <origin xyz="-0.032 0 0.070" rpy="0 0 0"/>
       <geometry>
-        <box size="0.140 0.140 0.143"/>
+        <cylinder radius="${collision_radius}" length="0.143" />
       </geometry>
     </collision>
@@ -41,8 +47,9 @@
     </inertial>
   </link>
+  <!-- Set the left wheel -->
   <joint name="${namespace}wheel_left_joint" type="continuous">
     <parent link="${namespace}base_link"/>
     <child link="${namespace}wheel_left_link"/>
-    <origin xyz="0.0 0.08 0.023" rpy="-1.57 0 0"/>
+    <origin xyz="0.0 ${track_width}/2 0.023" rpy="-1.57 0 0"/>
     <axis xyz="0 0 1"/>
   </joint>
@@ -53,10 +60,10 @@
         <mesh filename="package://nuturtle_description/meshes/left_tire.stl" scale="0.001 0.001 0.001"/>
       </geometry>
-      <material name="dark"/>
+      <material name="${color}"/>
     </visual>
     <collision>
       <origin xyz="0 0 0" rpy="0 0 0"/>
       <geometry>
-        <cylinder length="0.018" radius="0.033"/>
+        <cylinder length="0.018" radius="${wheel_radius}"/>
       </geometry>
     </collision>
@@ -67,8 +74,9 @@
     </inertial>
   </link>
+  <!-- Set the right wheel -->
   <joint name="${namespace}wheel_right_joint" type="continuous">
     <parent link="${namespace}base_link"/>
     <child link="${namespace}wheel_right_link"/>
-    <origin xyz="0.0 -0.080 0.023" rpy="-1.57 0 0"/>
+    <origin xyz="0.0 -${track_width}/2 0.023" rpy="-1.57 0 0"/>
     <axis xyz="0 0 1"/>
   </joint>
@@ -79,10 +87,10 @@
         <mesh filename="package://nuturtle_description/meshes/right_tire.stl" scale="0.001 0.001 0.001"/>
       </geometry>
-      <material name="dark"/>
+      <material name="${color}"/>
     </visual>
     <collision>
       <origin xyz="0 0 0" rpy="0 0 0"/>
       <geometry>
-        <cylinder length="0.018" radius="0.033"/>
+        <cylinder length="0.018" radius="${wheel_radius}"/>
       </geometry>
     </collision>
@@ -111,4 +119,5 @@
     </inertial>
   </link>
+  <!-- Set up the IMU -->
   <joint name="${namespace}imu_joint" type="fixed">
     <parent link="${namespace}base_link"/>
@@ -122,4 +131,5 @@
     <origin xyz="-0.032 0 0.172" rpy="0 0 0"/>
   </joint>
+  <!-- Set up the scanner -->
   <link name="${namespace}base_scan">
     <visual>
@@ -128,5 +138,5 @@
         <mesh filename="package://nuturtle_description/meshes/lds.stl" scale="0.001 0.001 0.001"/>
       </geometry>
-      <material name="dark"/>
+      <material name="${color}"/>
     </visual>
     <collision>

Commit message: Finished Task A.4. Removed the namespace argumenet from the urdf and changed it to set the namespace in the launchfile. Available colors are red, blue, green, and purple. Built and saved each load_one_color.rviz file fro the 4 colors. Did colocon test clean-up. Code passes all colcon tests! Next step is A.5.

File: nuturtle_description/urdf/common_properties.urdf.xacro (robot description, xacro)
@@ -15,4 +15,10 @@
     <color rgba="0.4 0.4 0.4 1.0"/>
   </material>
+  <material name="purple">
+    <color rgba="0.3 0.16 0.52 1.0"/>
+  </material>
+  <material name="red">
+    <color rgba="1.0 0.0 0.0 1.0"/>
+  </material>
   <material name="blue">
     <color rgba="0.0 0.0 0.8 1.0"/>
@@ -30,7 +36,4 @@
     <color rgba="${222/255} ${207/255} ${195/255} 1.0"/>
   </material>
-  <material name="red">
-    <color rgba="0.8 0.0 0.0 1.0"/>
-  </material>
   <material name="white">
     <color rgba="1.0 1.0 1.0 1.0"/>

File: nuturtle_description/urdf/turtlebot3_burger.urdf.xacro (robot description, xacro)
@@ -12,20 +12,12 @@
   <xacro:property name="track_width" value="${config['/**']['ros__parameters']['track_width']}"/>
   <xacro:property name="collision_radius" value="${config['/**']['ros__parameters']['collision_radius']}"/>
-  <!-- Define color property from Launch File -->
-  <!-- <xacro:property name="color" value="${config['/**']['ros__parameters']['color']}"/> -->
   <!--Load in the Xacros created to establish the colors of the nuturtle-->
   <xacro:include filename="$(find nuturtle_description)/urdf/common_properties.urdf.xacro"/>
-  <!-- Set the namespace of the robot -->
-  <xacro:arg name="namespace" default=""/>
-  <xacro:property name="namespace" value="$(arg namespace)"/>
+  <!-- Define color property from Launch File to set the color and namespace -->
+  <xacro:arg name="color" default="purple"/>
  <!-- Use the Xacros to build the URDF-->
-  <link name="${namespace}base_footprint"/>
-  <joint name="${namespace}base_joint" type="fixed">
-    <parent link="${namespace}base_footprint"/>
-    <child link="${namespace}base_link"/>
-    <origin xyz="0.0 0.0 0.010" rpy="0 0 0"/>
-  </joint>
+  <link name="base_footprint"/>
   <!-- Set the BaseLink -->
-  <link name="${namespace}base_link">
+  <link name="base_link">
     <visual>
       <origin xyz="-0.032 0 0.0" rpy="0 0 0"/>
@@ -33,5 +25,5 @@
         <mesh filename="package://nuturtle_description/meshes/burger_base.stl" scale="0.001 0.001 0.001"/>
       </geometry>
-      <material name="${color}"/>
+      <material name="$(arg color)"/>
     </visual>
     <collision>
@@ -47,12 +39,18 @@
     </inertial>
   </link>
+  <!-- Connect the footprint to the base_link -->
+  <joint name="base_joint" type="fixed">
+    <parent link="base_footprint"/>
+    <child link="base_link"/>
+    <origin xyz="0.0 0.0 0.010" rpy="0 0 0"/>
+  </joint>
   <!-- Set the left wheel -->
-  <joint name="${namespace}wheel_left_joint" type="continuous">
-    <parent link="${namespace}base_link"/>
-    <child link="${namespace}wheel_left_link"/>
-    <origin xyz="0.0 ${track_width}/2 0.023" rpy="-1.57 0 0"/>
+  <joint name="wheel_left_joint" type="continuous">
+    <parent link="base_link"/>
+    <child link="wheel_left_link"/>
+    <origin xyz="0.0 ${track_width/2} 0.023" rpy="-1.57 0 0"/>
     <axis xyz="0 0 1"/>
   </joint>
-  <link name="${namespace}wheel_left_link">
+  <link name="wheel_left_link">
     <visual>
       <origin xyz="0 0 0" rpy="1.57 0 0"/>
@@ -60,5 +58,5 @@
         <mesh filename="package://nuturtle_description/meshes/left_tire.stl" scale="0.001 0.001 0.001"/>
       </geometry>
-      <material name="${color}"/>
+      <material name="black"/>
     </visual>
     <collision>
@@ -75,11 +73,11 @@
   </link>
   <!-- Set the right wheel -->
-  <joint name="${namespace}wheel_right_joint" type="continuous">
-    <parent link="${namespace}base_link"/>
-    <child link="${namespace}wheel_right_link"/>
-    <origin xyz="0.0 -${track_width}/2 0.023" rpy="-1.57 0 0"/>
+  <joint name="wheel_right_joint" type="continuous">
+    <parent link="base_link"/>
+    <child link="wheel_right_link"/>
+    <origin xyz="0.0 ${-track_width/2} 0.023" rpy="-1.57 0 0"/>
     <axis xyz="0 0 1"/>
   </joint>
-  <link name="${namespace}wheel_right_link">
+  <link name="wheel_right_link">
     <visual>
       <origin xyz="0 0 0" rpy="1.57 0 0"/>
@@ -87,5 +85,5 @@
         <mesh filename="package://nuturtle_description/meshes/right_tire.stl" scale="0.001 0.001 0.001"/>
       </geometry>
-      <material name="${color}"/>
+      <material name="black"/>
     </visual>
     <collision>
@@ -101,10 +99,10 @@
     </inertial>
   </link>
-  <joint name="${namespace}caster_back_joint" type="fixed">
-    <parent link="${namespace}base_link"/>
-    <child link="${namespace}caster_back_link"/>
+  <joint name="caster_back_joint" type="fixed">
+    <parent link="base_link"/>
+    <child link="caster_back_link"/>
     <origin xyz="-0.081 0 -0.004" rpy="-1.57 0 0"/>
   </joint>
-  <link name="${namespace}caster_back_link">
+  <link name="caster_back_link">
     <collision>
       <origin xyz="0 0.001 0" rpy="0 0 0"/>
@@ -120,17 +118,17 @@
   </link>
   <!-- Set up the IMU -->
-  <joint name="${namespace}imu_joint" type="fixed">
-    <parent link="${namespace}base_link"/>
-    <child link="${namespace}imu_link"/>
+  <joint name="imu_joint" type="fixed">
+    <parent link="base_link"/>
+    <child link="imu_link"/>
     <origin xyz="-0.032 0 0.068" rpy="0 0 0"/>
   </joint>
-  <link name="${namespace}imu_link"/>
-  <joint name="${namespace}scan_joint" type="fixed">
-    <parent link="${namespace}base_link"/>
-    <child link="${namespace}base_scan"/>
+  <link name="imu_link"/>
+  <joint name="scan_joint" type="fixed">
+    <parent link="base_link"/>
+    <child link="base_scan"/>
     <origin xyz="-0.032 0 0.172" rpy="0 0 0"/>
   </joint>
   <!-- Set up the scanner -->
-  <link name="${namespace}base_scan">
+  <link name="base_scan">
     <visual>
       <origin xyz="0 0 0.0" rpy="0 0 0"/>
@@ -138,5 +136,5 @@
         <mesh filename="package://nuturtle_description/meshes/lds.stl" scale="0.001 0.001 0.001"/>
       </geometry>
-      <material name="${color}"/>
+      <material name="dark"/>
     </visual>
     <collision>
